File: NomiStar/NomiStar.kicad_pcb (KiCad board)
At the start: 2 copper layers, 120.1 x 88.7 mm, 12 parts, among them IC1 HT7833, J1 PINHD_1x4_Female, J2 PINHD_1x4_Female, J3 PINHD_1x4_Female, J4 PINHD_1x4_Female, J5 PINHD_1x4_Female, J6 Micro_SD_Card_Det1, J8 Conn_01x05, SW1 SW_Push, U1 STM32F373CBTx, U2 ESP32-S3-SuperMini

Commit message: Finished the pentagon board Need to design and draw up the point boards, maybe panelize it myself into small 2 boards
Parts:
- removed U2: ESP32-S3-SuperMini, ESP-super_mini:ESP32-S3-SuperMini
- added C10: 100 nF, Capacitor_SMD:C_0603_1608Metric, F.Cu at (82.4, 63.3)
- added J7: USB_C_Receptacle_USB2.0_16P, Connector_USB:USB_C_Receptacle_GCT_USB4105-xx-A_16P_TopMnt_Horizontal, B.Cu at (95.0, 103.3)
- added R10: 100, Resistor_SMD:R_0603_1608Metric, F.Cu at (90.1, 51.9)
- added R2: 5.1 k, Resistor_SMD:R_0603_1608Metric, F.Cu at (98.8, 95.5)
- added R3: 5.1 k, Resistor_SMD:R_0603_1608Metric, F.Cu at (88.5, 56.3)
- added R6: 5.1 k, Resistor_SMD:R_0603_1608Metric, F.Cu at (103.3, 59.3)
- added R7: 5.1 k, Resistor_SMD:R_0603_1608Metric, F.Cu at (114.6, 67.8)
- added R8: 5.1 k, Resistor_SMD:R_0603_1608Metric, F.Cu at (118.6, 67.8)
- added R9: 100, Resistor_SMD:R_0603_1608Metric, F.Cu at (81.7, 66.5)
- added REF**: NPTH, PCM_kikit:NPTH, F.Cu at (134.5, 86.4)
- added REF**: NPTH, PCM_kikit:NPTH, F.Cu at (121.6, 46.6)
- added REF**: NPTH, PCM_kikit:NPTH, F.Cu at (67.1, 86.3)
- added REF**: NPTH, PCM_kikit:NPTH, F.Cu at (121.2, 72.5)
- added REF**: NPTH, PCM_kikit:NPTH, F.Cu at (79.9, 46.6)
- added REF**: NPTH, PCM_kikit:NPTH, F.Cu at (100.8, 110.8)
- added REF**: NPTH, PCM_kikit:NPTH, F.Cu at (80.5, 72.5)
- added U3: ESP32-C3_SUPERMINI_TH, ESP-super_mini:MODULE_ESP32-C3_SUPERMINI_TH, F.Cu at (99.6, 83.6)
- IC1, J8, SW1: moved to B.Cu
- moved SW1 159.2 mm to (106.2, 102.0), turned to 180 degrees
- moved IC1 155.8 mm to (102.3, 95.3), turned to 180 degrees
- moved J5 148.4 mm to (72.4, 70.2), turned to 162 degrees
- moved J6 148.2 mm to (113.0, 58.0)
- moved R1 141.8 mm to (119.5, 77.6)
- moved J4 137.3 mm to (87.0, 100.8), turned to -126 degrees
- moved U1 114.2 mm to (90.0, 63.0)
- moved J8 111.7 mm to (100.8, 67.9), turned to 180 degrees
- moved J1 104.5 mm to (96.9, 46.8), turned to 90 degrees
- moved J3 100.4 mm to (120.7, 96.2), turned to -54 degrees
- moved J2 79.9 mm to (126.8, 62.9), turned to 18 degrees
Other:
- board size 120.1 x 88.7 mm -> 70.9 x 67.4 mm

Commit message: Finished the center PCB, will move onto the point schematic and PCB next
Parts:
- moved R1 35.0 mm to (94.1, 101.7)
Connections:
- J1 pad 3: +3.3V -> +5V
- J2 pad 3: +3.3V -> +5V
- J3 pad 3: +3.3V -> +5V
- J4 pad 3: +3.3V -> +5V
- J5 pad 3: +3.3V -> +5V
Routing:
- net +5V: track 0.00 -> 181.2 mm, vias 0 -> 8
- net +3.3V: track 0.00 -> 140.0 mm, vias 0 -> 14
- net Net-(U1-PA12): track 0.00 -> 71.5 mm, vias 0 -> 3
- net Net-(U1-PA10): track 0.00 -> 63.3 mm, vias 0 -> 6
- net Net-(U1-PA9): track 0.00 -> 58.7 mm, vias 0 -> 8
- net Net-(U1-PA2): track 0.00 -> 57.9 mm, vias 0 -> 1
- net Net-(J6-CMD): track 0.00 -> 55.5 mm, vias 0 -> 1
- net Net-(U1-PC13): track 0.00 -> 54.9 mm, vias 0 -> 5
- net Net-(U1-PA11): track 0.00 -> 52.8 mm, vias 0 -> 1
- net Net-(J6-DAT0): track 0.00 -> 51.4 mm, vias 0 -> 1
- net Net-(J6-DAT3/CD): track 0.00 -> 48.4 mm, vias 0 -> 2
- net Net-(U1-PA1): track 0.00 -> 46.6 mm, vias 0 -> 1
- net Net-(U3-GPIO1): track 0.00 -> 43.9 mm, vias 0 -> 2
- net Net-(J6-DET): track 0.00 -> 34.5 mm, vias 0 -> 1
- net Net-(J6-CLK): track 0.00 -> 33.7 mm
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- added copper zone on F.Cu, net GND
