File: NomiStar/NomiStarPoint/NomiStarPoint.kicad_pcb (KiCad board)
At the start: 2 copper layers, 75 x 43 mm, 13 parts, among them J1 Conn_01x04

Commit message: Fixed swapped data in and +5v
Connections:
- J1 pad 2: +5V -> Net-(D1-DIN)
- J1 pad 3: Net-(D1-DIN) -> +5V
Routing:
- net Net-(D1-DIN): track 21.6 -> 19.1 mm
Changed lines of the file:
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@@
 			)
 		)
-		(property "Description" ""
+		(property "Description" "Generic connector, single row, 01x04, script generated (kicad-library-utils/schlib/autogen/connector/)"
 			(at 0 0 0)
 			(layer "F.Fab")
@@
 		(sheetname "/")
 		(sheetfile "NomiStarPoint.kicad_sch")
+		(units
+			(unit
+				(name "A")
+				(pins "1" "2" "3" "4")
+			)
+		)
 		(attr through_hole)
 		(duplicate_pad_numbers_are_jumpers no)
@@
 			(layers "*.Cu" "*.Mask")
 			(remove_unused_layers no)
-			(net "+5V")
+			(net "Net-(D1-DIN)")
 			(pinfunction "Pin_2_2")
 			(pintype "passive")
@@
 			(layers "*.Cu" "*.Mask")
 			(remove_unused_layers no)
-			(net "Net-(D1-DIN)")
+			(net "+5V")
 			(pinfunction "Pin_3_3")
 			(pintype "passive")
@@
 	)
 	(segment
+		(start 51.9 82.4)
+		(end 51.8 82.3)
+		(width 0.2)
+		(layer "F.Cu")
+		(net "Net-(D8-DOUT)")
+	)
+	(segment
+		(start 59.7 82.4)
+		(end 51.9 82.4)
+		(width 0.2)
+		(layer "F.Cu")
+		(net "Net-(D8-DOUT)")
+	)
+	(segment
+		(start 85.05 67.1)
+		(end 87.15 69.2)
+		(width 0.2)
+		(layer "F.Cu")
+		(net "Net-(D4-DOUT)")
+	)
+	(segment
+		(start 87.15 69.2)
+		(end 101.05 69.2)
+		(width 0.2)
+		(layer "F.Cu")
+		(net "Net-(D4-DOUT)")
+	)
+	(segment
+		(start 101.05 69.2)
+		(end 102.65 67.6)
+		(width 0.2)
+		(layer "F.Cu")
+		(net "Net-(D4-DOUT)")
+	)
+	(segment
+		(start 88.15 65.6)
+		(end 74.4 65.6)
+		(width 0.2)
+		(layer "F.Cu")
+		(net "Net-(D3-DOUT)")
+	)
+	(segment
+		(start 74.4 65.6)
+		(end 72.35 63.55)
+		(width 0.2)
+		(layer "F.Cu")
+		(net "Net-(D3-DOUT)")
+	)
+	(segment
+		(start 89.95 63.8)
+		(end 88.15 65.6)
+		(width 0.2)
+		(layer "F.Cu")
+		(net "Net-(D3-DOUT)")
+	)
+	(via
+		(at 72.35 63.55)
+		(size 0.6)
+		(drill 0.3)
+		(layers "F.Cu" "B.Cu")
+		(net "Net-(D3-DOUT)")
+	)
+	(segment
+		(start 72.3 78.6)
+		(end 65.1 78.6)
+		(width 0.2)
+		(layer "F.Cu")
+		(net "Net-(D7-DOUT)")
+	)
+	(segment
+		(start 65.1 78.6)
+		(end 64.6 79.1)
+		(width 0.2)
+		(layer "F.Cu")
+		(net "Net-(D7-DOUT)")
+	)
+	(segment
+		(start 90.8 70.9)
+		(end 90 71.7)
+		(width 0.2)
+		(layer "F.Cu")
+		(net "Net-(D5-DOUT)")
+	)
+	(segment
+		(start 97.75 70.9)
+		(end 90.8 70.9)
+		(width 0.2)
+		(layer "F.Cu")
+		(net "Net-(D5-DOUT)")
+	)
+	(segment
+		(start 75.6 62)
+		(end 75.6 61.9)
+		(width 0.2)
+		(layer "F.Cu")
+		(net "Net-(D2-DOUT)")
+	)
+	(segment
+		(start 61.75 62)
+		(end 75.6 62)
+		(width 0.2)
+		(layer "F.Cu")
+		(net "Net-(D2-DOUT)")
+	)
+	(segment
+		(start 59.65 59.9)
+		(end 61.75 62)
+		(width 0.2)
+		(layer "F.Cu")
+		(net "Net-(D2-DOUT)")
+	)
+	(segment
+		(start 75.6 61.9)
+		(end 77.25 60.25)
+		(width 0.2)
+		(layer "F.Cu")
+		(net "Net-(D2-DOUT)")
+	)
+	(via
+		(at 46.95 56.25)
+		(size 0.6)
+		(drill 0.3)
+		(layers "F.Cu" "B.Cu")
+		(net "Net-(D1-DOUT)")
+	)
+	(via
+		(at 64.55 56.6)
+		(size 0.6)
+		(drill 0.3)
+		(layers "F.Cu" "B.Cu")
+		(net "Net-(D1-DOUT)")
+	)
+	(segment
+		(start 46.95 56.25)
+		(end 57.75 56.25)
+		(width 0.2)
+		(layer "B.Cu")
+		(net "Net-(D1-DOUT)")
+	)
+	(segment
+		(start 58.8 55.2)
+		(end 63.15 55.2)
+		(width 0.2)
+		(layer "B.Cu")
+		(net "Net-(D1-DOUT)")
+	)
+	(segment
+		(start 57.75 56.25)
+		(end 58.8 55.2)
+		(width 0.2)
+		(layer "B.Cu")
+		(net "Net-(D1-DOUT)")
+	)
+	(segment
+		(start 63.15 55.2)
+		(end 64.55 56.6)
+		(width 0.2)
+		(layer "B.Cu")
+		(net "Net-(D1-DOUT)")
+	)
+	(segment
 		(start 49.4 54.6)
 		(end 50.2 54.6)
@@
 	)
 	(segment
-		(start 49.4 64.87)
-		(end 49.4 54.6)
+		(start 49.4 54.6)
+		(end 49.4 62.33)
 		(width 0.2)
 		(layer "F.Cu")
@@
 	)
 	(segment
-		(start 43.6 70.67)
-		(end 49.4 64.87)
+		(start 49.4 62.33)
+		(end 43.6 68.13)
 		(width 0.2)
 		(layer "F.Cu")
 		(net "Net-(D1-DIN)")
-	)
-	(via
-		(at 46.95 56.25)
-		(size 0.6)
-		(drill 0.3)
-		(layers "F.Cu" "B.Cu")
-		(net "Net-(D1-DOUT)")
-	)
-	(via
-		(at 64.55 56.6)
-		(size 0.6)
-		(drill 0.3)
-		(layers "F.Cu" "B.Cu")
-		(net "Net-(D1-DOUT)")
-	)
-	(segment
-		(start 46.95 56.25)
-		(end 57.75 56.25)
-		(width 0.2)
-		(layer "B.Cu")
-		(net "Net-(D1-DOUT)")
-	)
-	(segment
-		(start 58.8 55.2)
-		(end 63.15 55.2)
-		(width 0.2)
-		(layer "B.Cu")
-		(net "Net-(D1-DOUT)")
-	)
-	(segment
-		(start 57.75 56.25)
-		(end 58.8 55.2)
-		(width 0.2)
-		(layer "B.Cu")
-		(net "Net-(D1-DOUT)")
-	)
-	(segment
-		(start 63.15 55.2)
-		(end 64.55 56.6)
-		(width 0.2)
-		(layer "B.Cu")
-		(net "Net-(D1-DOUT)")
-	)
-	(segment
-		(start 75.6 62)
-		(end 75.6 61.9)
-		(width 0.2)
-		(layer "F.Cu")
-		(net "Net-(D2-DOUT)")
-	)
-	(segment
-		(start 61.75 62)
-		(end 75.6 62)
-		(width 0.2)
-		(layer "F.Cu")
-		(net "Net-(D2-DOUT)")
-	)
-	(segment
-		(start 59.65 59.9)
-		(end 61.75 62)
-		(width 0.2)
-		(layer "F.Cu")
-		(net "Net-(D2-DOUT)")
-	)
-	(segment
-		(start 75.6 61.9)
-		(end 77.25 60.25)
-		(width 0.2)
-		(layer "F.Cu")
-		(net "Net-(D2-DOUT)")
-	)
-	(segment
-		(start 88.15 65.6)
-		(end 74.4 65.6)
-		(width 0.2)
-		(layer "F.Cu")
-		(net "Net-(D3-DOUT)")
-	)
-	(segment
-		(start 74.4 65.6)
-		(end 72.35 63.55)
-		(width 0.2)
-		(layer "F.Cu")
-		(net "Net-(D3-DOUT)")
-	)
-	(segment
-		(start 89.95 63.8)
-		(end 88.15 65.6)
-		(width 0.2)
-		(layer "F.Cu")
-		(net "Net-(D3-DOUT)")
-	)
-	(via
-		(at 72.35 63.55)
-		(size 0.6)
-		(drill 0.3)
-		(layers "F.Cu" "B.Cu")
-		(net "Net-(D3-DOUT)")
-	)
-	(segment
-		(start 85.05 67.1)
-		(end 87.15 69.2)
-		(width 0.2)
-		(layer "F.Cu")
-		(net "Net-(D4-DOUT)")
-	)
-	(segment
-		(start 87.15 69.2)
-		(end 101.05 69.2)
-		(width 0.2)
-		(layer "F.Cu")
-		(net "Net-(D4-DOUT)")
-	)
-	(segment
-		(start 101.05 69.2)
-		(end 102.65 67.6)
-		(width 0.2)
-		(layer "F.Cu")
-		(net "Net-(D4-DOUT)")
-	)
-	(segment
-		(start 90.8 70.9)
-		(end 90 71.7)
-		(width 0.2)
-		(layer "F.Cu")
-		(net "Net-(D5-DOUT)")
-	)
-	(segment
-		(start 97.75 70.9)
-		(end 90.8 70.9)
-		(width 0.2)
-		(layer "F.Cu")
-		(net "Net-(D5-DOUT)")
 	)
 	(segment
@@
 		(net "Net-(D6-DOUT)")
 	)
-	(segment
-		(start 72.3 78.6)
-		(end 65.1 78.6)
-		(width 0.2)
-		(layer "F.Cu")
-		(net "Net-(D7-DOUT)")
-	)
-	(segment
-		(start 65.1 78.6)
-		(end 64.6 79.1)
-		(width 0.2)
-		(layer "F.Cu")
-		(net "Net-(D7-DOUT)")
-	)
-	(segment
-		(start 51.9 82.4)
-		(end 51.8 82.3)
-		(width 0.2)
-		(layer "F.Cu")
-		(net "Net-(D8-DOUT)")
-	)
-	(segment
-		(start 59.7 82.4)
-		(end 51.9 82.4)
-		(width 0.2)
-		(layer "F.Cu")
-		(net "Net-(D8-DOUT)")
-	)
 	(zone
